Commit message: Create new pkg with my setup

File: Add/grippers/endoscope_attachment.xacro (robot description, xacro)
@@ -1,38 +1,43 @@
-<xacro:macro name="endoscope_camera" params="prefix parent">
-  <link name="${prefix}camera_link">
-    <inertial> ... </inertial>
-    <visual>
-      <geometry> <box size="0.05 0.03 0.03"/> </geometry>
-      <material name="blue"/>
-    </visual>
-  </link>
-  <joint name="${prefix}camera_joint" type="fixed">
-    <parent link="${parent}"/> <!-- es: gripper_center -->
-    <child link="${prefix}camera_link"/>
-    <origin xyz="0 0 -0.1" rpy="${-pi/2} 0 0"/> <!-- Assicura orientamento verso il target -->
-  </joint>
-  <!-- Plugin Gazebo per la camera -->
-  <gazebo reference="${prefix}camera_link">
-    <sensor type="camera" name="endoscope_cam">
-      <update_rate>30</update_rate>
-      <camera name="endoscope">
-        <horizontal_fov>1.0472</horizontal_fov> <!-- 60° -->
-        <image>
-          <width>640</width>
-          <height>480</height>
-          <format>R8G8B8</format>
-        </image>
-        <clip>
-          <near>0.1</near>
-          <far>100</far>
-        </clip>
-      </camera>
-      <plugin name="camera_controller" filename="libgazebo_ros_camera.so">
-        <ros>
-          <namespace>/endoscope</namespace>
-        </ros>
-        <frame_name>${prefix}camera_link</frame_name>
-      </plugin>
-    </sensor>
-  </gazebo>
-</xacro:macro>
+<?xml version="1.0"?>
+<robot xmlns:xacro="http://www.ros.org/wiki/xacro">
+  <xacro:macro name="endoscope_camera" params="prefix parent">
+    <link name="${prefix}camera_link">
+      <inertial> ... </inertial>
+      <visual>
+        <geometry>
+          <box size="0.05 0.03 0.03"/>
+        </geometry>
+        <material name="blue"/>
+      </visual>
+    </link>
+    <joint name="${prefix}camera_joint" type="fixed">
+      <parent link="${parent}"/> <!-- es: gripper_center -->
+      <child link="${prefix}camera_link"/>
+      <origin xyz="0 0 -0.1" rpy="${-pi/2} 0 0"/> <!-- Assicura orientamento verso il target -->
+    </joint>
+    <!-- Plugin Gazebo per la camera -->
+    <gazebo reference="${prefix}camera_link">
+      <sensor type="camera" name="endoscope_cam">
+        <update_rate>30</update_rate>
+        <camera name="endoscope">
+          <horizontal_fov>1.0472</horizontal_fov> <!-- 60° -->
+          <image>
+            <width>640</width>
+            <height>480</height>
+            <format>R8G8B8</format>
+          </image>
+          <clip>
+            <near>0.1</near>
+            <far>100</far>
+          </clip>
+        </camera>
+        <plugin name="camera_controller" filename="libgazebo_ros_camera.so">
+          <ros>
+            <namespace>/endoscope</namespace>
+          </ros>
+          <frame_name>${prefix}camera_link</frame_name>
+        </plugin>
+      </sensor>
+    </gazebo>
+  </xacro:macro>
+</robot>

File: Add/grippers/rg2_gripper.xacro (robot description, xacro)
@@ -1,19 +1,22 @@
-<xacro:macro name="rg2_gripper" params="prefix parent">
-  <link name="${prefix}gripper_base">
-    <visual>
-      <geometry>
-        <box size="0.09 0.03 0.02"/>
-      </geometry>
-      <material name="gray"/>
-    </visual>
-    <inertial>
-      <mass value="0.16"/>
-      <inertia ixx="1e-4" ixy="0" ixz="0" iyy="1e-4" iyz="0" izz="1e-4"/>
-    </inertial>
-  </link>
-  <joint name="${prefix}gripper_joint" type="fixed">
-    <parent link="${parent}"/>
-    <child link="${prefix}gripper_base"/>
-    <origin xyz="0 0 0.05" rpy="0 0 0"/>
-  </joint>
-</xacro:macro>
+<?xml version="1.0"?>
+<robot xmlns:xacro="http://www.ros.org/wiki/xacro">
+  <xacro:macro name="rg2_gripper" params="prefix parent">
+    <link name="${prefix}gripper_base">
+      <visual>
+        <geometry>
+          <box size="0.09 0.03 0.02"/>
+        </geometry>
+        <material name="gray"/>
+      </visual>
+      <inertial>
+        <mass value="0.16"/>
+        <inertia ixx="1e-4" ixy="0" ixz="0" iyy="1e-4" iyz="0" izz="1e-4"/>
+      </inertial>
+    </link>
+    <joint name="${prefix}gripper_joint" type="fixed">
+      <parent link="${parent}"/>
+      <child link="${prefix}gripper_base"/>
+      <origin xyz="0 0 0.05" rpy="0 0 0"/>
+    </joint>
+  </xacro:macro>
+</robot>

File: Add/ur3_gripper_endoscope.xacro (robot description, xacro)
@@ -1,66 +1,13 @@
 <?xml version="1.0"?>
-<robot xmlns:xacro="http://ros.org/wiki/xacro" name="ur3_gripper_endoscope">
+<robot xmlns:xacro="http://www.ros.org/wiki/xacro" name="ur3_gripper_endoscope">
   <!-- Robot base -->
   <xacro:include filename="$(find ur_description)/urdf/ur3.xacro"/>
-  <!-- MACRO del gripper: punta a un tuo xacro o quello della repo RG2 -->
-  <xacro:include filename="$(find my_ur3_setup)/urdf/rg2_gripper.xacro"/>
-  <!-- MACRO per la camera endoscopica -->
-  <xacro:macro name="endoscope_camera" params="prefix parent">
-    <link name="${prefix}camera_link">
-      <visual>
-        <origin xyz="0 0 0.04" rpy="0 0 0"/>
-        <geometry>
-          <cylinder radius="0.008" length="0.08"/>
-        </geometry>
-        <material name="blue">
-          <color rgba="0.1 0.3 0.7 1"/>
-        </material>
-      </visual>
-      <collision>
-        <origin xyz="0 0 0.04" rpy="0 0 0"/>
-        <geometry>
-          <cylinder radius="0.008" length="0.08"/>
-        </geometry>
-      </collision>
-      <inertial>
-        <origin xyz="0 0 0.04" rpy="0 0 0"/>
-        <mass value="0.01"/>
-        <inertia ixx="2e-5" iyy="2e-5" izz="1e-5" ixy="0" ixz="0" iyz="0"/>
-      </inertial>
-    </link>
-    <joint name="${prefix}camera_mount" type="fixed">
-      <parent link="${parent}"/>
-      <child link="${prefix}camera_link"/>
-      <origin xyz="0 0 0.08" rpy="0 0 0"/>
-    </joint>
-    <!-- Gazebo camera plugin -->
-    <gazebo reference="${prefix}camera_link">
-      <sensor type="camera" name="endoscope_cam">
-        <update_rate>30</update_rate>
-        <camera>
-          <horizontal_fov>1.0472</horizontal_fov>
-          <image>
-            <width>640</width>
-            <height>480</height>
-            <format>R8G8B8</format>
-          </image>
-          <clip>
-            <near>0.01</near>
-            <far>2</far>
-          </clip>
-        </camera>
-        <plugin name="camera_controller" filename="libgazebo_ros_camera.so">
-          <ros>
-            <namespace>/endoscope</namespace>
-          </ros>
-          <frame_name>${prefix}camera_link</frame_name>
-        </plugin>
-      </sensor>
-    </gazebo>
-  </xacro:macro>
-  <!-- Instanzia il gripper: -->
+  <!-- Include il gripper -->
+  <xacro:include filename="$(find my_ur3_setup)/urdf/grippers/rg2_gripper.xacro"/>
+  <!-- Include l'endoscopio -->
+  <xacro:include filename="$(find my_ur3_setup)/urdf/grippers/endoscope_attachment.xacro"/>
+  <!-- Instanzia il gripper -->
   <xacro:rg2_gripper prefix="endo_" parent="tool0"/>
-  <!-- Instanzia la camera sull’estremità del gripper: -->
-  <!-- Cambia "endo_gripper_base" su dove vuoi fissarlo (ad esempio tra le dita o sulla base) -->
+  <!-- Instanzia l'endoscopio camera sulla base del gripper -->
   <xacro:endoscope_camera prefix="endo_" parent="endo_gripper_base"/>
 </robot>

Commit message: ADD gripper and endo

File: Add/grippers/endoscope_attachment.xacro (robot description, xacro)
@@ -1,25 +1,36 @@
-<?xml version="1.0"?>
 <robot xmlns:xacro="http://www.ros.org/wiki/xacro">
+  <material name="blue">
+    <color rgba="0.1 0.1 0.8 1.0"/>
+  </material>
   <xacro:macro name="endoscope_camera" params="prefix parent">
     <link name="${prefix}camera_link">
-      <inertial> ... </inertial>
       <visual>
         <geometry>
-          <box size="0.05 0.03 0.03"/>
+          <cylinder length="0.12" radius="0.01"/>
         </geometry>
         <material name="blue"/>
       </visual>
+      <collision>
+        <geometry>
+          <cylinder length="0.12" radius="0.01"/>
+        </geometry>
+      </collision>
+      <inertial>
+        <mass value="0.05"/>
+        <origin xyz="0 0 0" rpy="0 0 0"/>
+        <inertia ixx="0.00001" ixy="0" ixz="0" iyy="0.00001" iyz="0" izz="0.00001"/>
+      </inertial>
     </link>
-    <joint name="${prefix}camera_joint" type="fixed">
-      <parent link="${parent}"/> <!-- es: gripper_center -->
+    <joint name="${prefix}fixed_joint" type="fixed">
+      <parent link="${parent}"/>
       <child link="${prefix}camera_link"/>
-      <origin xyz="0 0 -0.1" rpy="${-pi/2} 0 0"/> <!-- Assicura orientamento verso il target -->
+      <origin xyz="0 0 0.08" rpy="0 0 0"/>
     </joint>
-    <!-- Plugin Gazebo per la camera -->
+    <!-- Camera simulation per Gazebo -->
     <gazebo reference="${prefix}camera_link">
-      <sensor type="camera" name="endoscope_cam">
+      <sensor type="camera" name="${prefix}endoscope_cam">
         <update_rate>30</update_rate>
-        <camera name="endoscope">
-          <horizontal_fov>1.0472</horizontal_fov> <!-- 60° -->
+        <camera>
+          <horizontal_fov>1.0</horizontal_fov>
           <image>
             <width>640</width>
@@ -28,13 +39,13 @@
           </image>
           <clip>
-            <near>0.1</near>
-            <far>100</far>
+            <near>0.01</near>
+            <far>5</far>
           </clip>
         </camera>
-        <plugin name="camera_controller" filename="libgazebo_ros_camera.so">
-          <ros>
-            <namespace>/endoscope</namespace>
-          </ros>
-          <frame_name>${prefix}camera_link</frame_name>
+        <plugin name="gazebo_ros_camera" filename="libgazebo_ros_camera.so">
+          <robotNamespace>/</robotNamespace>
+          <frameName>${prefix}camera_link</frameName>
+          <cameraName>${prefix}endoscope_cam</cameraName>
+          <updateRate>30</updateRate>
         </plugin>
       </sensor>

File: Add/grippers/rg2_gripper.xacro (robot description, xacro)
@@ -1,21 +1,29 @@
-<?xml version="1.0"?>
 <robot xmlns:xacro="http://www.ros.org/wiki/xacro">
+  <material name="gray">
+    <color rgba="0.5 0.5 0.5 1.0"/>
+  </material>
   <xacro:macro name="rg2_gripper" params="prefix parent">
     <link name="${prefix}gripper_base">
       <visual>
         <geometry>
-          <box size="0.09 0.03 0.02"/>
+          <box size="0.05 0.03 0.02"/>
         </geometry>
         <material name="gray"/>
       </visual>
+      <collision>
+        <geometry>
+          <box size="0.05 0.03 0.02"/>
+        </geometry>
+      </collision>
       <inertial>
-        <mass value="0.16"/>
-        <inertia ixx="1e-4" ixy="0" ixz="0" iyy="1e-4" iyz="0" izz="1e-4"/>
+        <mass value="0.1"/>
+        <origin xyz="0 0 0" rpy="0 0 0"/>
+        <inertia ixx="0.0001" ixy="0" ixz="0" iyy="0.0001" iyz="0" izz="0.0001"/>
       </inertial>
     </link>
-    <joint name="${prefix}gripper_joint" type="fixed">
+    <joint name="${prefix}fixed_joint" type="fixed">
       <parent link="${parent}"/>
       <child link="${prefix}gripper_base"/>
-      <origin xyz="0 0 0.05" rpy="0 0 0"/>
+      <origin xyz="0 0 0.04" rpy="0 0 0"/>
     </joint>
   </xacro:macro>

File: Add/ur3_gripper_endoscope.xacro (robot description, xacro)
@@ -1,13 +1,13 @@
 <?xml version="1.0"?>
 <robot xmlns:xacro="http://www.ros.org/wiki/xacro" name="ur3_gripper_endoscope">
-  <!-- Robot base -->
+  <!-- Include modello base UR3: assicurati che il file base sia accessibile -->
   <xacro:include filename="$(find ur_description)/urdf/ur3.xacro"/>
-  <!-- Include il gripper -->
+  <!-- Includi macro gripper -->
   <xacro:include filename="$(find my_ur3_setup)/urdf/grippers/rg2_gripper.xacro"/>
-  <!-- Include l'endoscopio -->
+  <!-- Includi macro endoscopio -->
   <xacro:include filename="$(find my_ur3_setup)/urdf/grippers/endoscope_attachment.xacro"/>
-  <!-- Instanzia il gripper -->
-  <xacro:rg2_gripper prefix="endo_" parent="tool0"/>
-  <!-- Instanzia l'endoscopio camera sulla base del gripper -->
-  <xacro:endoscope_camera prefix="endo_" parent="endo_gripper_base"/>
+  <!-- Crea il gripper attaccato a tool0 -->
+  <xacro:rg2_gripper prefix="gripper_" parent="tool0"/>
+  <!-- Crea l'endoscopio/camera attaccato al gripper -->
+  <xacro:endoscope_camera prefix="endo_" parent="gripper_gripper_base"/>
 </robot>

Commit message: FIX endoscope dim

File: Add/grippers/endoscope_attachment.xacro (robot description, xacro)
@@ -1,23 +1,27 @@
 <robot xmlns:xacro="http://www.ros.org/wiki/xacro">
-  <material name="blue">
-    <color rgba="0.1 0.1 0.8 1.0"/>
+  <!-- Material definitions -->
+  <material name="metallic_silver">
+    <color rgba="0.7 0.7 0.7 1.0"/>
   </material>
+  <!-- Macro definition for the cystoscope camera -->
   <xacro:macro name="endoscope_camera" params="prefix parent">
     <link name="${prefix}camera_link">
       <visual>
         <geometry>
-          <cylinder length="0.12" radius="0.01"/>
+          <!-- Adjusting to typical dimensions: cylindrical length and diameter -->
+          <cylinder length="0.35" radius="0.004"/>
         </geometry>
-        <material name="blue"/>
+        <material name="metallic_silver"/>
       </visual>
       <collision>
         <geometry>
-          <cylinder length="0.12" radius="0.01"/>
+          <cylinder length="0.35" radius="0.004"/>
         </geometry>
       </collision>
       <inertial>
-        <mass value="0.05"/>
+        <mass value="0.1"/>
         <origin xyz="0 0 0" rpy="0 0 0"/>
-        <inertia ixx="0.00001" ixy="0" ixz="0" iyy="0.00001" iyz="0" izz="0.00001"/>
+        <!-- Adjusted inertia values -->
+        <inertia ixx="0.000005" ixy="0" ixz="0" iyy="0.000005" iyz="0" izz="0.000005"/>
       </inertial>
     </link>
@@ -25,20 +29,21 @@
       <parent link="${parent}"/>
       <child link="${prefix}camera_link"/>
-      <origin xyz="0 0 0.08" rpy="0 0 0"/>
+      <origin xyz="0 0 0.18" rpy="0 0 0"/>
     </joint>
-    <!-- Camera simulation per Gazebo -->
+    <!-- Camera simulation enhancements for Gazebo -->
     <gazebo reference="${prefix}camera_link">
       <sensor type="camera" name="${prefix}endoscope_cam">
         <update_rate>30</update_rate>
         <camera>
-          <horizontal_fov>1.0</horizontal_fov>
+          <!-- Improved field of view and resolution -->
+          <horizontal_fov>1.57</horizontal_fov> <!-- 90 degrees (in radians) -->
           <image>
-            <width>640</width>
-            <height>480</height>
+            <width>1920</width> <!-- Higher resolution -->
+            <height>1080</height>
             <format>R8G8B8</format>
           </image>
           <clip>
             <near>0.01</near>
-            <far>5</far>
+            <far>10</far>
           </clip>
         </camera>

Commit message: Fix endo-tip

File: Add/grippers/endoscope_attachment.xacro (robot description, xacro)
@@ -1,43 +1,125 @@
 <robot xmlns:xacro="http://www.ros.org/wiki/xacro">
   <!-- Material definitions -->
-  <material name="metallic_silver">
-    <color rgba="0.7 0.7 0.7 1.0"/>
+  <material name="metallic_white">
+    <color rgba="1.0 1.0 1.0 1.0"/>
   </material>
-  <!-- Macro definition for the cystoscope camera -->
+  <material name="camera_red">
+    <color rgba="1.0 0.0 0.0 1.0"/>
+  </material>
+  <!-- Macro definition for the endoscope with angled tip -->
   <xacro:macro name="endoscope_camera" params="prefix parent">
+    <!-- Main endoscope shaft - straight part -->
+    <link name="${prefix}shaft_link">
+      <visual>
+        <geometry>
+          <cylinder length="0.33" radius="0.004"/>
+        </geometry>
+        <origin xyz="0 0 0" rpy="0 0 0"/>
+        <material name="metallic_white"/>
+      </visual>
+      <collision>
+        <geometry>
+          <cylinder length="0.33" radius="0.004"/>
+        </geometry>
+        <origin xyz="0 0 0" rpy="0 0 0"/>
+      </collision>
+      <inertial>
+        <mass value="0.08"/>
+        <origin xyz="0 0 0" rpy="0 0 0"/>
+        <inertia ixx="0.000004" ixy="0" ixz="0" iyy="0.000004" iyz="0" izz="0.000004"/>
+      </inertial>
+    </link>
+    <!-- Connect to parent link -->
+    <joint name="${prefix}shaft_joint" type="fixed">
+      <parent link="${parent}"/>
+      <child link="${prefix}shaft_link"/>
+      <origin xyz="0 0 0.18" rpy="0 0 0"/>
+    </joint>
+    <!-- Angled tip (45-degree cut) -->
+    <link name="${prefix}angled_tip">
+      <visual>
+        <!-- Using a mesh would be ideal here, but for simplicity, we'll use a box that's rotated -->
+        <geometry>
+          <box size="0.005 0.005 0.005"/>
+        </geometry>
+        <!-- Position at the tip of the shaft and rotate to create 45-degree angle effect -->
+        <origin xyz="0 0 0" rpy="0 ${pi/4} 0"/>
+        <material name="metallic_white"/>
+      </visual>
+      <collision>
+        <geometry>
+          <box size="0.005 0.005 0.005"/>
+        </geometry>
+        <origin xyz="0 0 0" rpy="0 ${pi/4} 0"/>
+      </collision>
+      <inertial>
+        <mass value="0.001"/>
+        <origin xyz="0 0 0" rpy="0 ${pi/4} 0"/>
+        <inertia ixx="0.0000001" ixy="0" ixz="0" iyy="0.0000001" iyz="0" izz="0.0000001"/>
+      </inertial>
+    </link>
+    <!-- Joint connecting angled tip to shaft -->
+    <joint name="${prefix}tip_joint" type="fixed">
+      <parent link="${prefix}shaft_link"/>
+      <child link="${prefix}angled_tip"/>
+      <!-- Position at the end of the shaft -->
+      <origin xyz="0 0 0.165" rpy="0 0 0"/>
+    </joint>
+    <!-- Camera link - positioned at the angled tip -->
     <link name="${prefix}camera_link">
       <visual>
         <geometry>
-          <!-- Adjusting to typical dimensions: cylindrical length and diameter -->
-          <cylinder length="0.35" radius="0.004"/>
+          <sphere radius="0.0015"/>
         </geometry>
-        <material name="metallic_silver"/>
+        <material name="camera_red"/>
       </visual>
       <collision>
         <geometry>
-          <cylinder length="0.35" radius="0.004"/>
+          <sphere radius="0.0015"/>
         </geometry>
       </collision>
       <inertial>
-        <mass value="0.1"/>
-        <origin xyz="0 0 0" rpy="0 0 0"/>
-        <!-- Adjusted inertia values -->
-        <inertia ixx="0.000005" ixy="0" ixz="0" iyy="0.000005" iyz="0" izz="0.000005"/>
+        <mass value="0.002"/>
+        <origin xyz="-0.005 0 0" rpy="0 ${-pi/4} 0"/>
+        <inertia ixx="0.00000005" ixy="0" ixz="0" iyy="0.00000005" iyz="0" izz="0.00000005"/>
       </inertial>
     </link>
-    <joint name="${prefix}fixed_joint" type="fixed">
-      <parent link="${parent}"/>
+    <!-- Joint placing camera at the angled tip, oriented at 45 degrees -->
+    <joint name="${prefix}camera_joint" type="fixed">
+      <parent link="${prefix}angled_tip"/>
       <child link="${prefix}camera_link"/>
-      <origin xyz="0 0 0.18" rpy="0 0 0"/>
+      <!-- Position camera at the center of the angled face -->
+      <origin xyz="0 0 0.003" rpy="0 ${pi/4} 0"/>
     </joint>
-    <!-- Camera simulation enhancements for Gazebo -->
+    <!-- Camera indicator (optional, for visibility) -->
+    <link name="${prefix}camera_direction">
+      <visual>
+        <geometry>
+          <cylinder length="0.005" radius="0.0005"/>
+        </geometry>
+        <material name="camera_red"/>
+      </visual>
+      <inertial>
+        <mass value="0.0001"/>
+        <origin xyz="0 0 0" rpy="0 0 0"/>
+        <inertia ixx="0.00000001" ixy="0" ixz="0" iyy="0.00000001" iyz="0" izz="0.00000001"/>
+      </inertial>
+    </link>
+    <!-- Joint for camera direction indicator -->
+    <joint name="${prefix}camera_direction_joint" type="fixed">
+      <parent link="${prefix}camera_link"/>
+      <child link="${prefix}camera_direction"/>
+      <!-- Position in front of camera, pointing outward -->
+      <origin xyz="0 0 0.0025" rpy="0 0 0"/>
+    </joint>
+    <!-- Gazebo camera setup -->
     <gazebo reference="${prefix}camera_link">
-      <sensor type="camera" name="${prefix}endoscope_cam">
+      <material>Gazebo/Red</material>
+      <sensor type="camera" name="${prefix}endoscope_camera">
         <update_rate>30</update_rate>
         <camera>
-          <!-- Improved field of view and resolution -->
-          <horizontal_fov>1.57</horizontal_fov> <!-- 90 degrees (in radians) -->
+          <horizontal_fov>1.57</horizontal_fov>
           <image>
-            <width>1920</width> <!-- Higher resolution -->
+            <width>1920</width>
             <height>1080</height>
             <format>R8G8B8</format>
@@ -51,6 +133,12 @@
           <robotNamespace>/</robotNamespace>
           <frameName>${prefix}camera_link</frameName>
-          <cameraName>${prefix}endoscope_cam</cameraName>
+          <cameraName>${prefix}endoscope_camera</cameraName>
           <updateRate>30</updateRate>
+          <hackBaseline>0.07</hackBaseline>
+          <distortionK1>0.0</distortionK1>
+          <distortionK2>0.0</distortionK2>
+          <distortionK3>0.0</distortionK3>
+          <distortionT1>0.0</distortionT1>
+          <distortionT2>0.0</distortionT2>
         </plugin>
       </sensor>
