Commit message: Renamed and cleaned

File: Add/endoscope.xacro (robot description, xacro)
@@ -70,5 +70,5 @@
       <visual>
         <geometry>
-          <sphere radius="0.0015"/>
+          <sphere radius="0.0005"/>
         </geometry>
         <material name="camera_red"/>
@@ -76,5 +76,5 @@
       <collision>
         <geometry>
-          <sphere radius="0.0015"/>
+          <sphere radius="0.0005"/>
         </geometry>
       </collision>
@@ -91,25 +91,4 @@
       <!-- Position camera at the center of the angled face -->
       <origin xyz="0 0 0.003" rpy="0 ${pi/4} 0"/>
-    </joint>
-    <!-- Camera indicator (optional, for visibility) -->
-    <link name="${prefix}camera_direction">
-      <visual>
-        <geometry>
-          <cylinder length="0.005" radius="0.0005"/>
-        </geometry>
-        <material name="camera_red"/>
-      </visual>
-      <inertial>
-        <mass value="0.0001"/>
-        <origin xyz="0 0 0" rpy="0 0 0"/>
-        <inertia ixx="0.00000001" ixy="0" ixz="0" iyy="0.00000001" iyz="0" izz="0.00000001"/>
-      </inertial>
-    </link>
-    <!-- Joint for camera direction indicator -->
-    <joint name="${prefix}camera_direction_joint" type="fixed">
-      <parent link="${prefix}camera_link"/>
-      <child link="${prefix}camera_direction"/>
-      <!-- Position in front of camera, pointing outward -->
-      <origin xyz="0 0 0.0025" rpy="0 0 0"/>
     </joint>
     <!-- Gazebo camera setup -->

File: Add/ur.xacro (robot description, xacro)
@@ -2,7 +2,6 @@
   <!-- Include macro per il robot UR -->
   <xacro:include filename="$(find ur_gazebo)/urdf/ur_macro.xacro"/>
-  <!-- Include macro per il gripper e l'endoscopio -->
-  <xacro:include filename="$(find my_ur3_setup)/urdf/grippers/rg2_gripper.xacro"/>
-  <xacro:include filename="$(find my_ur3_setup)/urdf/grippers/endoscope_attachment.xacro"/>
+  <!-- Include macro per l'endoscopio -->
+  <xacro:include filename="$(find my_ur3_setup)/urdf/endoscope.xacro"/>
   <!-- Parametri dichiarati dall'utente -->
   <xacro:arg name="joint_limit_params" default=""/>
@@ -26,8 +25,6 @@
     safety_k_position="$(arg safety_k_position)"
   />
-  <!-- Aggiungi il gripper al tool0 -->
-  <xacro:rg2_gripper prefix="gripper_" parent="tool0"/>
   <!-- Aggiungi l'endoscopio montato sul gripper -->
-  <xacro:endoscope_camera prefix="endo_" parent="gripper_gripper_base"/>
+  <xacro:endoscope_camera prefix="endo_" parent="tool0"/>
   <!-- Fissare la base del robot al mondo -->
   <link name="world"/>
@@ -37,5 +34,5 @@
     <origin xyz="0 0 0" rpy="0 0 0"/>
   </joint>
-  <!-- Interfaccia per controller (facoltativa) -->
+    <!-- Interfaccia per controller (facoltativa) -->
   <link name="tool0_controller"/>
   <joint name="tool_controller_fake_joint" type="fixed">
