Commit message: Fix coordinate of joins and links

File: ADD/ur3_endoscope_description/urdf/endoscope.xacro (robot description, xacro)
@@ -1,38 +1,35 @@
 <?xml version="1.0"?>
 <robot xmlns:xacro="http://www.ros.org/wiki/xacro">
-  <xacro:macro name="endoscope" params="parent_link xyz rpy"> <!-- Aggiunti xyz e rpy come parametri -->
-    <!-- Corpo principale dell'endoscopio -->
+  <xacro:macro name="endoscope" params="parent_link xyz rpy">
+    <!-- Corpo principale dell'endoscopio (più corto e grosso) -->
     <link name="endoscope_body_link">
       <visual>
         <geometry>
-          <cylinder length="0.39" radius="0.005"/> <!-- Primo cilindro -->
+          <cylinder length="0.13" radius="0.025"/> <!-- Corpo corto e grosso -->
         </geometry>
         <material name="blue"/>
       </visual>
     </link>
-    <!-- Punta dell'endoscopio -->
+    <!-- Punta dell'endoscopio (stretta e lunga) -->
     <link name="endoscope_tip_link">
       <visual>
         <geometry>
-          <cylinder length="0.13" radius="0.025"/> <!-- Secondo cilindro -->
+          <cylinder length="0.39" radius="0.005"/> <!-- Punta stretta e lunga -->
         </geometry>
-        <!-- L'origine del visual all'interno del link. Mantengo come era, ma potrebbe richiedere aggiustamenti visivi. -->
-        <origin xyz="0 0 0.26" rpy="0 0 0"/>
+        <origin xyz="0 0 0.195" rpy="0 0 0"/> <!-- Offset per connettere al corpo -->
         <material name="blue"/>
       </visual>
     </link>
-    <!-- Joint collegando l'endoscopio al gripper -->
-    <!-- L'origine di questo joint è ora definita dai parametri xyz e rpy passati alla macro. -->
+    <!-- Joint che collega l'endoscopio al gripper -->
     <joint name="${parent_link}_endoscope_joint" type="fixed">
-      <origin xyz="${xyz}" rpy="${rpy}"/> <!-- Usa i parametri passati -->
+      <origin xyz="${xyz}" rpy="${rpy}"/>
       <parent link="${parent_link}"/>
       <child link="endoscope_body_link"/>
     </joint>
-    <!-- Joint collegando il corpo dell'endoscopio alla punta -->
-    <!-- Questo joint è interno all'endoscopio e non cambia. -->
+    <!-- Joint che collega il corpo alla punta -->
     <joint name="endoscope_tip_joint" type="fixed">
       <parent link="endoscope_body_link"/>
       <child link="endoscope_tip_link"/>
-      <origin xyz="0 0 0.195" rpy="0 0 0"/> <!-- Offset della punta rispetto al corpo dell'endoscopio -->
+      <origin xyz="0 0 0" rpy="0 0 0"/> <!-- Connesso più vicino alla punta -->
     </joint>
   </xacro:macro>

File: ADD/ur3_endoscope_description/urdf/gripper.xacro (robot description, xacro)
@@ -14,5 +14,5 @@
     <!-- L'origine xyz="0 0 0" rpy="0 0 0" posiziona il gripper rispetto al parent link. -->
     <joint name="${parent_link}_gripper_joint" type="fixed">
-      <origin xyz="0.0375 0 0" rpy="0 1.5708 0"/>
+      <origin xyz="0 0 0.06" rpy="0 0 1.5708"/>
       <parent link="${parent_link}"/>
       <child link="gripper_base_link"/>

File: ADD/ur3_endoscope_description/urdf/ur3_endoscope.urdf.xacro (robot description, xacro)
@@ -135,5 +135,5 @@
    <!-- Rotazione: rpy="0 1.5708 0" (pitch di 90 gradi) fa sì che l'endoscopio punti in avanti lungo l'asse X del gripper. -->
    <!-- Spostamento: xyz="-0.195 0 0" sposta l'origine del link del corpo dell'endoscopio indietro di 0.195 lungo il suo asse X (che ora è l'asse Z originale ruotato), in modo che la punta (a +0.195 lungo l'asse Z originale) si trovi all'origine del gripper. -->
-   <xacro:endoscope parent_link="gripper_base_link" xyz="-0.195 0 0" rpy="0 1.5708 0"/>
+   <xacro:endoscope parent_link="gripper_base_link" xyz="-0.1025 0 0.095" rpy="0 1.5708 0"/>
    <!-- === ADDED GRIPPER AND ENDOSCOPE END === -->
    <xacro:if value="$(arg sim_gazebo)">

Commit message: ADD collision

File: ADD/ur3_endoscope_description/urdf/endoscope.xacro (robot description, xacro)
@@ -10,4 +10,9 @@
         <material name="blue"/>
       </visual>
+      <collision>
+        <geometry>
+          <cylinder length="0.13" radius="0.025"/> <!-- Corpo collisione uguale a quella visiva -->
+        </geometry>
+      </collision>
     </link>
     <!-- Punta dell'endoscopio (stretta e lunga) -->
@@ -20,4 +25,10 @@
         <material name="blue"/>
       </visual>
+      <collision>
+        <geometry>
+          <cylinder length="0.39" radius="0.005"/> <!-- Corpo collisione uguale a quella visiva -->
+        </geometry>
+        <origin xyz="0 0 0.195" rpy="0 0 0"/> <!-- Stesso offset della parte visiva -->
+      </collision>
     </link>
     <!-- Joint che collega l'endoscopio al gripper -->

File: ADD/ur3_endoscope_description/urdf/gripper.xacro (robot description, xacro)
@@ -6,13 +6,18 @@
       <visual>
         <geometry>
-          <box size="0.075 0.075 0.19"/> <!-- Dimensioni generiche del gripper -->
+          <box size="0.075 0.075 0.18"/> <!-- Dimensioni generiche del gripper -->
         </geometry>
         <material name="grey"/>
       </visual>
+      <collision>
+        <geometry>
+          <box size="0.075 0.075 0.18"/> <!-- Geometria di collisione uguale a quella visiva -->
+        </geometry>
+      </collision>
     </link>
     <!-- Joint collegando il gripper al link parent (wrist_3_link) -->
     <!-- L'origine xyz="0 0 0" rpy="0 0 0" posiziona il gripper rispetto al parent link. -->
     <joint name="${parent_link}_gripper_joint" type="fixed">
-      <origin xyz="0 0 0.06" rpy="0 0 1.5708"/>
+      <origin xyz="0 0 0.09" rpy="0 0 1.5708"/>
       <parent link="${parent_link}"/>
       <child link="gripper_base_link"/>

File: ADD/ur3_endoscope_description/urdf/ur3_endoscope.urdf.xacro (robot description, xacro)
@@ -1,11 +1,11 @@
 <?xml version="1.0"?>
-<robot xmlns:xacro="http://wiki.ros.org/xacro" name="$(arg name)">
+<robot xmlns:xacro="http://wiki.ros.org/xacro" name="ur3">
    <!-- robot name parameter -->
-   <xacro:arg name="name" default="ur"/>
+   <xacro:arg name="name" default="ur3"/>
    <!-- import main macro -->
    <xacro:include filename="$(find ur_description)/urdf/ur_macro.xacro"/>
    <!-- possible 'ur_type' values: ur3, ur3e, ur5, ur5e, ur7e, ur10, ur10e, ur12e, ur16e, ur15, ur20, ur30 -->
    <!-- the default value should raise an error in case this was called without defining the type -->
-   <xacro:arg name="ur_type" default="ur5x"/>
+   <xacro:arg name="ur_type" default="ur3"/>
    <!-- DEFINIZIONI DEI MATERIALI QUI -->
    <material name="grey">
@@ -86,5 +86,5 @@
    <!-- arm -->
    <xacro:ur_robot
-     name="$(arg name)"
+     name="ur3"
      tf_prefix="$(arg tf_prefix)"
      parent="world"

Commit message: Fix some dimension in urdf model

File: ADD/ur3_endoscope_description/urdf/endoscope.xacro (robot description, xacro)
@@ -42,5 +42,5 @@
       <parent link="endoscope_body_link"/>
       <child link="endoscope_tip_link"/>
-      <origin xyz="0 0 0" rpy="0 0 0"/> <!-- Connesso più vicino alla punta -->
+      <origin xyz="0 0 0.065" rpy="0 0 0"/> <!-- Connesso più vicino alla punta -->
     </joint>
   </xacro:macro>

File: ADD/ur3_endoscope_description/urdf/gripper.xacro (robot description, xacro)
@@ -6,5 +6,5 @@
       <visual>
         <geometry>
-          <box size="0.075 0.075 0.18"/> <!-- Dimensioni generiche del gripper -->
+          <box size="0.075 0.075 0.24"/> <!-- Dimensioni generiche del gripper -->
         </geometry>
         <material name="grey"/>
@@ -12,5 +12,5 @@
       <collision>
         <geometry>
-          <box size="0.075 0.075 0.18"/> <!-- Geometria di collisione uguale a quella visiva -->
+          <box size="0.075 0.075 0.24"/> <!-- Geometria di collisione uguale a quella visiva -->
         </geometry>
       </collision>

File: ADD/ur3_endoscope_description/urdf/ur3_endoscope.urdf.xacro (robot description, xacro)
@@ -135,5 +135,5 @@
    <!-- Rotazione: rpy="0 1.5708 0" (pitch di 90 gradi) fa sì che l'endoscopio punti in avanti lungo l'asse X del gripper. -->
    <!-- Spostamento: xyz="-0.195 0 0" sposta l'origine del link del corpo dell'endoscopio indietro di 0.195 lungo il suo asse X (che ora è l'asse Z originale ruotato), in modo che la punta (a +0.195 lungo l'asse Z originale) si trovi all'origine del gripper. -->
-   <xacro:endoscope parent_link="gripper_base_link" xyz="-0.1025 0 0.095" rpy="0 1.5708 0"/>
+   <xacro:endoscope parent_link="gripper_base_link" xyz="-0.1025 0 0.12" rpy="0 1.5708 0"/>
    <!-- === ADDED GRIPPER AND ENDOSCOPE END === -->
    <xacro:if value="$(arg sim_gazebo)">

Commit message: ADD eng comments

File: ADD/ur3_endoscope_description/urdf/endoscope.xacro (robot description, xacro)
@@ -1,10 +1,11 @@
 <?xml version="1.0"?>
 <robot xmlns:xacro="http://www.ros.org/wiki/xacro">
+<!-- This section defines the endoscope model (body and tip), as used in the robot system. -->
   <xacro:macro name="endoscope" params="parent_link xyz rpy">
-    <!-- Corpo principale dell'endoscopio (più corto e grosso) -->
+    <!-- Main body of the endoscope (shorter and thicker) -->
     <link name="endoscope_body_link">
       <visual>
         <geometry>
-          <cylinder length="0.13" radius="0.025"/> <!-- Corpo corto e grosso -->
+          <cylinder length="0.13" radius="0.025"/> <!-- Short and thick body -->
         </geometry>
         <material name="blue"/>
@@ -12,25 +13,25 @@
       <collision>
         <geometry>
-          <cylinder length="0.13" radius="0.025"/> <!-- Corpo collisione uguale a quella visiva -->
+          <cylinder length="0.13" radius="0.025"/> <!-- Collision body same as visual -->
         </geometry>
       </collision>
     </link>
-    <!-- Punta dell'endoscopio (stretta e lunga) -->
+    <!-- Tip of the endoscope (thin and long) -->
     <link name="endoscope_tip_link">
       <visual>
         <geometry>
-          <cylinder length="0.39" radius="0.005"/> <!-- Punta stretta e lunga -->
+          <cylinder length="0.39" radius="0.005"/> <!-- Thin and long tip -->
         </geometry>
-        <origin xyz="0 0 0.195" rpy="0 0 0"/> <!-- Offset per connettere al corpo -->
+        <origin xyz="0 0 0.195" rpy="0 0 0"/> <!-- Offset to connect to the body -->
         <material name="blue"/>
       </visual>
       <collision>
         <geometry>
-          <cylinder length="0.39" radius="0.005"/> <!-- Corpo collisione uguale a quella visiva -->
+          <cylinder length="0.39" radius="0.005"/> <!-- Collision body same as visual -->
         </geometry>
-        <origin xyz="0 0 0.195" rpy="0 0 0"/> <!-- Stesso offset della parte visiva -->
+        <origin xyz="0 0 0.195" rpy="0 0 0"/> <!-- Same offset as the visual part -->
       </collision>
     </link>
-    <!-- Joint che collega l'endoscopio al gripper -->
+    <!-- Joint connecting the endoscope to the gripper -->
     <joint name="${parent_link}_endoscope_joint" type="fixed">
       <origin xyz="${xyz}" rpy="${rpy}"/>
@@ -38,9 +39,9 @@
       <child link="endoscope_body_link"/>
     </joint>
-    <!-- Joint che collega il corpo alla punta -->
+    <!-- Joint connecting the body to the tip -->
     <joint name="endoscope_tip_joint" type="fixed">
       <parent link="endoscope_body_link"/>
       <child link="endoscope_tip_link"/>
-      <origin xyz="0 0 0.065" rpy="0 0 0"/> <!-- Connesso più vicino alla punta -->
+      <origin xyz="0 0 0.065" rpy="0 0 0"/> <!-- Connected tip to tip -->
     </joint>
   </xacro:macro>

File: ADD/ur3_endoscope_description/urdf/gripper.xacro (robot description, xacro)
@@ -1,10 +1,13 @@
 <?xml version="1.0"?>
 <robot xmlns:xacro="http://www.ros.org/wiki/xacro">
+  <!--
+    This macro defines a simple gripper model to be attached to the robot.
+  -->
   <xacro:macro name="gripper" params="parent_link">
-    <!-- Gripper link -->
+    <!-- Gripper body -->
     <link name="gripper_base_link">
       <visual>
         <geometry>
-          <box size="0.075 0.075 0.24"/> <!-- Dimensioni generiche del gripper -->
+          <box size="0.075 0.075 0.24"/>
         </geometry>
         <material name="grey"/>
@@ -12,10 +15,10 @@
       <collision>
         <geometry>
-          <box size="0.075 0.075 0.24"/> <!-- Geometria di collisione uguale a quella visiva -->
+          <box size="0.075 0.075 0.24"/> <!-- Collision geometry same as visual -->
         </geometry>
       </collision>
     </link>
-    <!-- Joint collegando il gripper al link parent (wrist_3_link) -->
-    <!-- L'origine xyz="0 0 0" rpy="0 0 0" posiziona il gripper rispetto al parent link. -->
+    <!-- Joint connecting the gripper to the parent link (wrist_3_link) -->
+    <!-- The origin xyz="0 0 0.09" rpy="0 0 90deg" positions the gripper relative to the parent link. -->
     <joint name="${parent_link}_gripper_joint" type="fixed">
       <origin xyz="0 0 0.09" rpy="0 0 1.5708"/>

File: ADD/ur3_endoscope_description/urdf/ur3_endoscope.urdf.xacro (robot description, xacro)
@@ -8,10 +8,10 @@
    <!-- the default value should raise an error in case this was called without defining the type -->
    <xacro:arg name="ur_type" default="ur3"/>
-   <!-- DEFINIZIONI DEI MATERIALI QUI -->
+   <!-- Definition of materials -->
    <material name="grey">
-     <color rgba="0.7 0.7 0.7 1.0"/> <!-- Grigio medio opaco -->
+     <color rgba="0.7 0.7 0.7 1.0"/>
    </material>
    <material name="blue">
-     <color rgba="0.0 0.0 0.8 1.0"/> <!-- Blu scuro opaco -->
+     <color rgba="0.0 0.0 0.8 1.0"/>
    </material>
    <!-- parameters -->
@@ -125,16 +125,15 @@
    </xacro:ur_robot>
    <!-- === ADDED GRIPPER AND ENDOSCOPE START === -->
-   <!-- Inclusione dei file delle macro per gripper ed endoscopio -->
+   <!-- Inclusion of macro files for gripper and endoscope -->
    <xacro:include filename="$(find ur3_endoscope_description)/urdf/gripper.xacro"/>
    <xacro:include filename="$(find ur3_endoscope_description)/urdf/endoscope.xacro"/>
-   <!-- Gripper: attaccato al wrist_3_link del braccio robotico -->
-   <!-- La macro gripper.xacro definirà l'origine del gripper rispetto al suo parent_link. -->
-   <xacro:gripper parent_link="wrist_3_link"/>
-   <!-- Endoscopio: attaccato al gripper_base_link -->
-   <!-- Posizionamento: La sua origine è definita per posizionare la fine del corpo dell'endoscopio (dove si attacca la punta) sull'origine del gripper_base_link. -->
-   <!-- Rotazione: rpy="0 1.5708 0" (pitch di 90 gradi) fa sì che l'endoscopio punti in avanti lungo l'asse X del gripper. -->
-   <!-- Spostamento: xyz="-0.195 0 0" sposta l'origine del link del corpo dell'endoscopio indietro di 0.195 lungo il suo asse X (che ora è l'asse Z originale ruotato), in modo che la punta (a +0.195 lungo l'asse Z originale) si trovi all'origine del gripper. -->
-   <xacro:endoscope parent_link="gripper_base_link" xyz="-0.1025 0 0.12" rpy="0 1.5708 0"/>
-   <!-- === ADDED GRIPPER AND ENDOSCOPE END === -->
+   <!-- Gripper: attached to the wrist_3_link of the robotic arm -->
+   <!-- The gripper.xacro macro will define the gripper's origin relative to its parent_link. -->
+  <xacro:gripper parent_link="wrist_3_link"/>
+  <!-- Endoscope: Attached to gripper_base_link -->
+  <!-- Positioning: Its origin is defined to position the end of the endoscope body (where the tip attaches) at the origin of the gripper_base_link. -->
+  <!-- Rotation: rpy="0 1.5708 0" (90-degree pitch) causes the endoscope to point forward along the gripper's X-axis. -->
+  <!-- Displacement: xyz="-0.1025 0 12" moves the endoscope body's link origin back 0.1025 along its X-axis (which is now the original rotated Z-axis), so that the tip (at +0.1025 along the original Z-axis) is at the gripper's origin. -->
+  <xacro:endoscope parent_link="gripper_base_link" xyz="-0.1025 0 0.12" rpy="0 1.5708 0"/>
    <xacro:if value="$(arg sim_gazebo)">
     <!-- Gazebo plugins -->
